File: SenseWing/10DOF_FeatherWing.sch (EAGLE design)
At the start: 15 parts

Commit message: added v5 SenseWing
Parts:
- removed FC5: 0.1uF, SparkFun-Capacitors:0.1UF-25V(+80/-20%)(0603)
- removed FLASH: S25FL127SABMFI101, memory-spansion:S25FL127SABMFI101
- removed R_SCL, R_SDA: 4.7K, SparkFun-Resistors:4.7KOHM-1/10W-1%(0603)
- removed R_SW: 10K, SparkFun-Resistors:10KOHM-1/10W-1%(0603)0603
- added RC1: 100nf, Seeed-OPL-Capacitor:CERAMIC-100NF-50V-10%-X7R(0603)
- added RC2: 4.7uf, Seeed-OPL-Capacitor:CERAMIC-4.7UF-10V-10%-X5R(0603)
- added RSCL, RSDA: 4.7K, Seeed-OPL-Resistor:SMD-RES-4.7K-5%-1/10W(0603)
- added RSW: 10K, Seeed-OPL-Resistor:SMD-RES-10K-1%-1/10W(0603)
- added SRV_H2: (no value), SparkFun-Connectors:M03PTH
- added U$1: VL53L0X, VL53L0X:VL53L0X
- EC3, EC4, XC1, XC2: value 0.1uF -> 100nf; device SparkFun-Capacitors:0.1UF-25V(+80/-20%)(0603) -> Seeed-OPL-Capacitor:CERAMIC-100NF-50V-10%-X7R(0603)
- S1: value SWITCH-MOMENTARY-2SMD -> B3U-1000P; device SparkFun-Electromechanical:SWITCH-MOMENTARY-2SMD -> Seeed-OPL-Button:SMD-BUTTON-WITHOUT-BOSS-(2P-3X2.5MM)
Connections:
- net #0_RED_BL: now also U$1.XSHUT
- net #15_PD_BL: no longer FLASH.!CS!
- net #2_BLUE_PU_BL: now also SRV_H2.3
- net 3.3V: now also RC1.1, RC2.2, RSCL.2, RSDA.2, RSW.1, U$1.AVDD, U$1.AVDDVCSEL; no longer FC5.1, FLASH.VCC, R_SCL.2, R_SDA.2, R_SW.1
- net GND: now also RC1.2, RC2.1, SRV_H2.1, U$1.AVSSVCSEL, U$1.GND, U$1.GND@2, U$1.GND@3, U$1.GND@4; no longer FC5.2, FLASH.VSS
- net MISO: no longer FLASH.SO/IO1
- net MOSI: no longer FLASH.IO0/SI
- net SCK: no longer FLASH.SCK
- net SCL: now also RSCL.1, U$1.SCL; no longer R_SCL.1
- net SDA: now also RSDA.1, U$1.SDA; no longer R_SDA.1
- net SW1: now also RSW.2; no longer R_SW.2
- net VBAT: now also SRV_H2.2
Other:
- note added: "MPU9250 DECOUPLING"
- note added: "VL53L0X DECOUPLING"
- note removed: "BMX055 DECOUPLING"
- note removed: "FLASH"
- note removed: "FLASH DECOUPLING"
- moved on the sheet: BMX055
